File: 0012_GSM_GPS_Module_SIM800C.kicad_sch (KiCad schematic)
At the start: 25 parts, among them J1 sim, Q1 S8050, Q2 S8050, U1 SIM800C

Commit message: Add files via upload
Parts:
- added C1: 10uF, Capacitor_Tantalum_SMD:CP_EIA-2012-12_Kemet-R, symbol Device:C_Polarized_Small_US
- added C2: 22uF, Capacitor_SMD:C_0603_1608Metric, symbol Device:C_Small
- added D4: LED, LED_SMD:LED_0603_1608Metric, symbol Device:LED
- added J2: 20279-001E-01, L-KLS1-IPEX-20279-001E-0:L-KLS1-IPEX-20279-001E-0, symbol L-KLS1-IPEX-20279-001E-0:20279-001E-01
- added R11: R, Resistor_SMD:R_0603_1608Metric, symbol Device:R
- added R12: 220r, Resistor_SMD:R_0603_1608Metric, symbol Device:R
- added R13: 100r, Resistor_SMD:R_0603_1608Metric, symbol Device:R
- added U2: ~, Moduler_:pin_header_5-3, symbol moduler_pin:air
- added U3: MIC29302AWD, Package_TO_SOT_SMD:TO-252-5_TabPin3, symbol Regulator_Linear:MIC29302AWD
- C10, C11, C4, C5, C6, C7, C8, C9: footprint (none) -> Capacitor_SMD:C_0603_1608Metric
- D1: footprint (none) -> Diode_SMD:D_0603_1608Metric
- D2: footprint (none) -> LED_SMD:LED_0603_1608Metric
- D3: footprint SC70-6 -> SMF05C:SC70-6
- J1: footprint LKLS1SIM06462PH185R -> sim:LKLS1SIM06462PH185R
- Q1, Q2: footprint Package_TO_SOT_THT:TO-92_Inline -> Package_TO_SOT_SMD:SOT-23
- R1, R10, R2, R3, R4, R5, R6, R7, R8, R9: footprint (none) -> Resistor_SMD:R_0603_1608Metric
Connections:
- net CLK_EN: now also D3.5; no longer D3.1
- net D1: now also U2.12
- net DATA_EN: now also D3.4; no longer D3.5
- net GND: now also C1.2, C2.2, D4.1 (K), J2.2, J2.3, R13.2, U2.9, U3.3 (GND)
- net RST_EN: now also D3.1; no longer D3.4
- net RX: now also U2.11
- net TX: now also U2.10
- net at U1.32 (GSM_ANT): now also J2.1
- net VCC renamed +4V
- net +4V: now also C2.1, R12.1, U3.4 (VOUT)
- new net: R12.2, R13.1, U3.5 (ADJ)
- new net: D4.2 (A), R11.2
- new net +5V: C1.1, R11.1, U2.7, U3.1 (EN), U3.2 (VIN)
- no-connect marks 27 -> 40
Other:
- note added: "AIR PIN"
- note added: "BUCK"
- note added: "SENSOR"
- note added: "SIM CARD"
- moved on the sheet: C10, C11, C8, C9, D3, J1, R1, R2, R3
